File: 001_Sin-Resistencias/MakerCozumel.kicad_pcb (KiCad board)
At the start: 2 copper layers, 60.3 x 54.2 mm, 10 parts, among them SW1 SW_SPDT

Commit message: Some updates
Parts:
- added svg2mod: G***, Cozumel:Cu.In.03, F.Cu at (121.4, 89.8)
- REF**: moved to F.Cu
- moved REF** 1.27 mm to (138.4, 99.7)
Changed lines of the file:
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@@
-(kicad_pcb (version 20171130) (host pcbnew 6.0.0-rc1-unknown-5b3202d~66~ubuntu16.04.1)
+(kicad_pcb (version 20171130) (host pcbnew 5.0.2-bee76a0~70~ubuntu16.04.1)
   (general
     (thickness 1.6)
@@
     (tracks 27)
     (zones 0)
-    (modules 10)
+    (modules 11)
     (nets 4)
   )
@@
   )
   (layers
-    (0 F.Cu signal)
+    (0 F.Cu signal hide)
     (31 B.Cu signal)
     (34 B.Paste user)
@@
     (zone_45_only no)
     (trace_min 0.1524)
+    (segment_width 0.1524)
+    (edge_width 0.1524)
     (via_size 0.6858)
     (via_drill 0.3302)
@@
     (uvia_min_size 0)
     (uvia_min_drill 0)
-    (edge_width 0.1524)
-    (segment_width 0.1524)
     (pcb_text_width 0.1524)
     (pcb_text_size 1.016 1.016)
@@
     (mod_text_size 1.016 1.016)
     (mod_text_width 0.1524)
-    (pad_size 1.524 1.524)
-    (pad_drill 0.762)
+    (pad_size 5 5)
+    (pad_drill 0)
     (pad_to_mask_clearance 0.0762)
     (solder_mask_min_width 0.1016)
@@
       (xy -13.043149 0.887065)) (layer B.SilkS) (width 0))
   )
-  (module Cozumel:Pin2_Badge (layer B.Cu)
-    (at 138.43 98.425 180)
-    (fp_text reference REF** (at 0 -7.62 180) (layer B.Fab)
-      (effects (font (size 1 1) (thickness 0.15)) (justify mirror))
-    )
-    (fp_text value Pin2_Badge (at 0 7.9248 180) (layer B.Fab)
-      (effects (font (size 1 1) (thickness 0.15)) (justify mirror))
-    )
-    (pad 1 smd circle (at 0 0 180) (size 4 4) (layers B.Cu B.Paste B.Mask))
+  (module Cozumel:Pin2_Badge (layer F.Cu)
+    (at 138.43 99.695 180)
+    (fp_text reference REF** (at 0 7.62 180) (layer F.Fab)
+      (effects (font (size 1 1) (thickness 0.15)))
+    )
+    (fp_text value Pin2_Badge (at 0 -7.9248 180) (layer F.Fab)
+      (effects (font (size 1 1) (thickness 0.15)))
+    )
+    (pad 1 smd circle (at 0 0 180) (size 5 5) (layers B.Cu B.Paste B.Mask))
   )
   (module Cozumel:Ment.All.03 (layer F.Cu)
@@
     (fp_line (start 15.992359 27.026845) (end 15.269822 26.954824) (layer Edge.Cuts) (width 0.264375))
   )
+  (module Cozumel:Cu.In.03 (layer F.Cu)
+    (at 121.412 89.8398)
+    (descr "Imported from Ment.svg")
+    (tags svg2mod)
+    (attr smd)
+    (fp_text reference svg2mod (at 0 -7.722186) (layer F.SilkS) hide
+      (effects (font (size 1.524 1.524) (thickness 0.3048)))
+    )
+    (fp_text value G*** (at 0 7.722186) (layer F.SilkS) hide
+      (effects (font (size 1.524 1.524) (thickness 0.3048)))
+    )
+    (fp_poly (pts (xy -4.409044 4.674186) (xy -3.294365 4.674186) (xy -2.179686 4.674186) (xy -1.065005 4.674186)
+      (xy 0.049676 4.674186) (xy 1.164356 4.674186) (xy 2.279037 4.674186) (xy 3.393718 4.674186)
+      (xy 4.508398 4.674186) (xy 4.76111 4.661873) (xy 5.007166 4.625773) (xy 5.473982 4.487218)
+      (xy 5.8982 4.268533) (xy 6.269168 3.979736) (xy 6.57535 3.63084) (xy 6.80166 3.231866)
+      (xy 6.932118 2.792827) (xy 6.950747 2.323738) (xy 6.943652 1.769513) (xy 6.936557 1.215287)
+      (xy 6.929462 0.661062) (xy 6.922367 0.106837) (xy 6.915272 -0.447388) (xy 6.908177 -1.001613)
+      (xy 6.901082 -1.555838) (xy 6.893987 -2.110063) (xy 6.884236 -2.301203) (xy 6.8585 -2.47732)
+      (xy 6.822115 -2.643421) (xy 6.780403 -2.804512) (xy 6.579055 -3.20693) (xy 6.319799 -3.56991)
+      (xy 6.008624 -3.889069) (xy 5.651522 -4.160026) (xy 5.254483 -4.378398) (xy 4.823499 -4.539803)
+      (xy 4.364558 -4.63986) (xy 3.883652 -4.674186) (xy 2.910969 -4.674186) (xy 1.938286 -4.674186)
+      (xy 0.965603 -4.674186) (xy -0.007079 -4.674186) (xy -0.979762 -4.674186) (xy -1.952445 -4.674186)
+      (xy -2.925127 -4.674186) (xy -3.89781 -4.674186) (xy -4.518828 -4.615863) (xy -5.095914 -4.447989)
+      (xy -5.617089 -4.181206) (xy -6.070371 -3.826156) (xy -6.443781 -3.39348) (xy -6.725335 -2.893822)
+      (xy -6.903054 -2.337823) (xy -6.964957 -1.736126) (xy -6.943658 -1.215288) (xy -6.922358 -0.694451)
+      (xy -6.901059 -0.173613) (xy -6.87976 0.347224) (xy -6.85846 0.868062) (xy -6.837161 1.3889)
+      (xy -6.815862 1.909739) (xy -6.794562 2.430577) (xy -6.747969 2.895074) (xy -6.613514 3.322011)
+      (xy -6.399187 3.703875) (xy -6.112974 4.033154) (xy -5.762861 4.302337) (xy -5.356838 4.503911)
+      (xy -4.902889 4.630365) (xy -4.409004 4.674186) (xy -4.409025 4.674186) (xy -4.409044 4.674186)) (layer F.Cu) (width 0))
+  )
   (gr_text "Designed\nby" (at 139.0142 119.5832) (layer B.SilkS)
